File: eagle/maymusicbox.brd (EAGLE design)
At the start: 55.6 x 41.3 mm, 39 parts, among them CN1 BATT, Q1 IRF9530

Commit message: Fix Schematic + Part to have 0 error issues
Parts:
- MP3DIS: device 74xx-us:DIL20 -> May Music Box Parts:DIL20
Changed lines of the file:
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@@
 <attribute name="VALUE" x="42.418" y="32.893" size="1.27" layer="27" ratio="10" rot="R180"/>
 </element>
-<element name="MP3DIS" library="74xx-us" package="DIL20" value="74LS541N" x="19.9" y="15.968" smashed="yes" rot="R270">
+<element name="MP3DIS" library="May Music Box Parts" package="DIL20" value="74LS541N" x="19.9" y="15.968" smashed="yes" rot="R270">
 <attribute name="NAME" x="20.662" y="12.539" size="1.27" layer="25" rot="R90"/>
 </element>
